Commit message: modified:   arm_config/setup.py 	modified:   arm_description/urdf/OpenArmVKillian.xacro

File: arm_description/urdf/OpenArmVKillian.xacro (robot description, xacro)
@@ -7,5 +7,5 @@
     <link name="Cycloidal_Simplified_for_FEA">
         <inertial>
-            <origin xyz="-0.010005039449546161 4.037251654477103e-05 -0.031015874921037394" rpy=" -0.0 0.0" />
+            <origin xyz="-0.010005039449546161 4.037251654477103e-05 -0.031015874921037394" rpy="0.0 -0.0 0.0" />
             <mass value="0.43211727572229136" />
             <inertia ixx="0.0004211761261660727" iyy="0.00041859561398810397" izz="0.00039046053891583755" ixy="4.2155668701638026e-07" iyz="6.3117373221706e-07" ixz="-1.0981594307291016e-05" />
