Commit message: fixing stuff

File: arm_description/urdf/AmigoArmControl.xacro (robot description, xacro)
@@ -1,5 +1,5 @@
 <?xml version="1.0"?>
 <robot name="Amigo_Arm" xmlns:xacro="http://www.ros.org/wiki/xacro">
-  <xacro:macro name="Amigo_Arm_Control">
+  <xacro:macro name="AmigoArmControl">
     <!--4 DOF Arm-->
     <ros2_control name="arm_4DOF" type="system">
@@ -9,5 +9,5 @@
       </hardware>
       <joint name="joint1">
-        <param name="can_id">0</param>
+        <param name="can_id">1</param>
         <param name="pole_pairs">14</param>
         <param name="gear_ratio">36</param>
@@ -25,5 +25,5 @@
       </joint>
       <joint name="joint2">
-        <param name="can_id">1</param>
+        <param name="can_id">2</param>
         <param name="pole_pairs">14</param>
         <param name="gear_ratio">36</param>
@@ -41,5 +41,5 @@
       </joint>
       <joint name="joint3">
-        <param name="can_id">2</param>
+        <param name="can_id">3</param>
         <param name="pole_pairs">14</param>
         <param name="gear_ratio">36</param>

Commit message: fixing service call

File: arm_description/urdf/AmigoArmControl.xacro (robot description, xacro)
@@ -1,10 +1,10 @@
 <?xml version="1.0"?>
 <robot name="Amigo_Arm" xmlns:xacro="http://www.ros.org/wiki/xacro">
-  <xacro:macro name="AmigoArmControl">
+  <xacro:macro name="AmigoArmControl" params="hardware_plugin:='cubemars_hardware/CubeMarsSystemHardware' can_interface:='can0'">
     <!--4 DOF Arm-->
     <ros2_control name="arm_4DOF" type="system">
       <hardware>
-        <plugin>cubemars_hardware/CubeMarsSystemHardware</plugin>
-        <param name="can_interface">can0</param>
+        <plugin>${hardware_plugin}</plugin>
+        <param name="can_interface">${can_interface}</param>
       </hardware>
       <joint name="joint1">
